Commit message: [update] objects_models and panda robot to make every object pick-able

File: scibotpark/objects_models/ycb_objects/YcbChipsCan/model.urdf (robot description, URDF)
Before this commit: robot model.urdf, 1 links, 0 joints
Links:
- link baseLink: mass .205 -> .0205

File: scibotpark/objects_models/ycb_objects/YcbCrackerBox/model.urdf (robot description, URDF)
Before this commit: robot model.urdf, 1 links, 0 joints
Links:
- link baseLink: mass .411 -> .0411

File: scibotpark/objects_models/ycb_objects/YcbHammer/model.urdf (robot description, URDF)
Before this commit: robot model.urdf, 1 links, 0 joints
Links:
- link baseLink: mass .665 -> .065

File: scibotpark/objects_models/ycb_objects/YcbMasterChefCan/model.urdf (robot description, URDF)
Before this commit: robot model.urdf, 1 links, 0 joints
Links:
- link baseLink: mass .404 -> .0404

File: scibotpark/objects_models/ycb_objects/YcbMustardBottle/model.urdf (robot description, URDF)
Before this commit: robot model.urdf, 1 links, 0 joints
Links:
- link baseLink: mass .603 -> .303

File: scibotpark/objects_models/ycb_objects/YcbPowerDrill/model.urdf (robot description, URDF)
Before this commit: robot model.urdf, 1 links, 0 joints
Links:
- link baseLink: mass .895 -> .195
